File: Piggyback_1_0_PCB/Piggyback_1_0_PCB.kicad_pcb (KiCad board)
At the start: 2 copper layers, 52.4 x 19 mm, 39 parts, among them J10 Conn_02x04_Odd_Even, J11 Conn_02x04_Odd_Even, J12 Conn_01x04_Female, J13 Conn_01x04_Female, J2 Conn_02x04_Odd_Even, J3 Conn_01x04_Female, J4 Conn_02x04_Odd_Even, J5 Conn_01x04_Female, J6 Conn_01x04_Female, J7 Conn_01x04_Female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

Commit message: 1.0 commit
Parts:
- moved G*** 0.81 mm to (85.7, 81.8)
Other:
- board text added: "github.com/NCKiser/Piggyback_1.0"
Changed lines of the file:
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@@
     )
     (pad_to_mask_clearance 0)
-    (grid_origin 83.975 83.34375)
+    (grid_origin 85.725 76.2)
     (pcbplotparams
       (layerselection 0x00010fc_ffffffff)
@@
   )
   (footprint "LOGO" (layer "B.Cu")
-    (at 85.5625 80.9625 180)
+    (at 85.725 81.75625 180)
     (attr board_only exclude_from_pos_files exclude_from_bom)
     (fp_text reference "G***" (at 0 0) (layer "B.SilkS") hide
@@
   (gr_line (start 97.63125 78.58125) (end 102.39375 83.34375) (layer "Edge.Cuts") (width 0.05))
   (gr_line (start 92.86875 78.58125) (end 92.86875 69.05625) (layer "Edge.Cuts") (width 0.05))
+  (gr_text "github.com/NCKiser/Piggyback_1.0" (at 85.725 85.725) (layer "B.SilkS")
+    (effects (font (size 1.5 1.2) (thickness 0.25)) (justify mirror))
+  )
   (gr_text "D+ D-" (at 109.694408 86.171253 270) (layer "F.SilkS")
     (effects (font (size 1 0.6) (thickness 0.15)))

Commit message: Public commit
Other:
- board text added: "github.com/NCKiser/Piggyback"
- board text removed: "github.com/NCKiser/Piggyback_1.0"
Changed lines of the file:
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@@
   (gr_line (start 97.63125 78.58125) (end 102.39375 83.34375) (layer "Edge.Cuts") (width 0.05))
   (gr_line (start 92.86875 78.58125) (end 92.86875 69.05625) (layer "Edge.Cuts") (width 0.05))
-  (gr_text "github.com/NCKiser/Piggyback_1.0" (at 85.725 85.725) (layer "B.SilkS")
-    (effects (font (size 1.5 1.2) (thickness 0.25)) (justify mirror))
+  (gr_text "github.com/NCKiser/Piggyback" (at 85.725 85.725) (layer "B.SilkS")
+    (effects (font (size 1.5 1.4) (thickness 0.25)) (justify mirror))
   )
   (gr_text "D+ D-" (at 109.694408 86.171253 270) (layer "F.SilkS")

Commit message: Connected NC pads to GND and 5V
Connections:
- J11 pad 3: Net-(J11-Pad3) -> VCC
- J11 pad 4: Net-(J11-Pad4) -> GND
- J13 pad 3: Net-(J11-Pad3) -> VCC
- J9 pad 2: Net-(J11-Pad4) -> GND
- U1 pad 3: unconnected-(U1-Pad3) -> GND
- U1 pad 4: unconnected-(U1-Pad4) -> +5V
Routing:
- net GND: track 101.2 -> 106.0 mm, vias 18 -> 19
- net VCC: track 9.99 -> 13.9 mm
- net UCAP: track 16.6 -> 17.9 mm
- net C7: track 19.2 -> 18.4 mm
Other:
- board text added: "6A"
- board text removed: "6"
- board text removed: "AREF"

Commit message: More material around edge vias, no longer "castellated"
Routing:
- net +5V: track 88.3 -> 87.5 mm, vias 17 -> 14
- net D6: track 20.2 -> 19.8 mm, vias 2 -> 1
- net C6: track 21.9 -> 21.5 mm, vias 2 -> 1
- net B5: track 21.2 -> 20.8 mm, vias 3 -> 2
- net B1: track 17.3 -> 16.9 mm, vias 2 -> 1
- net D--: track 11.0 -> 10.6 mm, vias 3 -> 2
- net GND: track 106.0 -> 105.6 mm, vias 19 -> 18
- net UCAP: vias 3 -> 2
- net D7: vias 2 -> 1
- net D4: vias 2 -> 1
- net D++: vias 3 -> 2
- net C7: vias 2 -> 1
- net B6: vias 3 -> 2
- net B4: vias 2 -> 1
- net B2: vias 2 -> 1
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Other:
- board size 52.4 x 19 mm -> 52.4 x 19.2 mm
