File: PiggybackBT_1_0/PiggybackBT_1_0.kicad_pcb (KiCad board)
At the start: 4 copper layers, 63.5 x 26.2 mm, 53 parts, among them J1 Conn_02x04_Odd_Even, J2 Conn_02x04_Odd_Even, J3 Conn_02x04_Odd_Even, J4 Conn_02x04_Odd_Even, J5 Conn_01x02, U1 BQ24075/9, U2 SRV05-4, U3 nRF52840, Y1 32.768 kHz, Y2 32MHz

Commit message: Minor Updates
Parts:
- removed REF** (x4): breakaway-mousebites, Keebio-Parts:breakaway-mousebites
Connections:
- J4 pad 4: unconnected-(J4-Pad4) -> GND
- U3 pad U1: P0.12 -> unconnected-(U3-PadU1)
Routing:
- net GND: track 122.2 -> 125.7 mm
- net P0.12: track 0.68 -> 0.00 mm, vias 1 -> 0
