File: PiggybackBT_1_0/PiggybackBT_1_0.kicad_sch (KiCad schematic)
At the start: 49 parts, among them J1 Conn_02x04_Odd_Even, J2 Conn_02x04_Odd_Even, J3 Conn_02x04_Odd_Even, J4 Conn_02x04_Odd_Even, J5 Conn_01x02, U1 BQ24075/9, U2 SRV05-4, U3 nRF52840, Y1 32.768 kHz, Y2 32MHz

Commit message: Minor Updates
Connections:
- net GND: now also J4.4 (Pin_4)
- net P0.12: no longer names the net of U3.U1 (TRACEDATA1/P0.12)
- net P0.13: no longer names the net of U3.AD8 (P0.13)
