File: Piggyback_2_0/Piggyback_2_0.kicad_pcb (KiCad board)
At the start: 2 copper layers, 93.7 x 55.6 mm, 54 parts, among them J1 USB_C_Receptacle_USB2.0, J2 Conn_01x14_Female, J3 Conn_01x06_Female, J4 Conn_01x14_Female, J5 Conn_01x06_Female, J6 Conn_01x04_Male, J7 Conn_01x05_Female, SW1 MX_SW_solder, SW10 MX_SW_solder, SW11 MX_SW_solder, SW12 MX_SW_solder, SW13 MX_SW_solder, SW14 MX_SW_solder, SW15 MX_SW_solder, SW2 MX_SW_solder, SW3 MX_SW_solder, SW4 MX_SW_solder, SW5 MX_SW_solder, SW6 MX_SW_solder, SW7 MX_SW_solder, SW8 MX_SW_solder, SW9 MX_SW_solder, U1 RP2040TR7, U2 XC6206PxxxMR, U3 SRV05-4, U4 W25Q128JVS, Y1 Crystal_GND24_Small

Commit message: made a lot of changes
Parts:
- removed the C10 at (164.5, 92.7)
- removed the C12 at (175.4, 104.8)
- removed J4: Conn_01x14_Female, Connector_PinHeader_2.54mm:PinHeader_1x14_P2.54mm_Vertical
- removed J6: Conn_01x04_Male, Connector_JST:JST_SH_SM04B-SRSS-TB_1x04-1MP_P1.00mm_Horizontal
- removed J7: Conn_01x05_Female, Connector_PinHeader_2.54mm:PinHeader_1x05_P2.54mm_Vertical
- removed SW4: MX_SW_solder, marbastlib-mx:SW_MX_1u
- added D1: D_Small, Diode_SMD:D_SOD-123, B.Cu at (99.2, 90.5)
- added D2: D_Small, Diode_SMD:D_SOD-123, B.Cu at (108.7, 90.5)
- added D3: D_Small, Diode_SMD:D_SOD-123, B.Cu at (127.8, 90.5)
- added EZ1: 78171-0004, locallib:PicoEZMate-Reinforced-Lite, B.Cu at (118.8, 76.4)
- added G***: LOGO, LOGO, F.Cu at (88.9, 77.8)
- added G***: LOGO, LOGO, F.Cu at (107.2, 84.1)
- added REF**: mousebites 2mm, marbastlib-various:mousebites_2mm, F.Cu at (127.8, 73.9)
- J1: value USB_C_Receptacle_USB2.0 -> Conn_01x06_Female; footprint Connector_USB:USB_C_Receptacle_HRO_TYPE-C-31-M-12 -> Connector_PinHeader_2.54mm:PinHeader_1x06_P2.54mm_Vertical; moved to F.Cu
- J2: value Conn_01x14_Female -> Conn_01x23_Female; footprint Connector_PinHeader_2.54mm:PinHeader_1x14_P2.54mm_Vertical -> Connector_PinHeader_2.54mm:PinHeader_1x22_P2.54mm_Vertical; moved to B.Cu
- J3: value Conn_01x06_Female -> USB_C_Receptacle_USB2.0; footprint Connector_PinHeader_2.54mm:PinHeader_1x06_P2.54mm_Vertical -> Connector_USB:USB_C_Receptacle_HRO_TYPE-C-31-M-12; moved to B.Cu
- R1, R2: value R_Small -> 5.1k
- moved R3 118.2 mm to (87.3, 76.2), turned to 90 degrees
- moved R6 112.7 mm to (92.9, 86.5), turned to 45 degrees
- moved SWR1 100.2 mm to (84.1, 76.2), turned to 0 degrees
- moved Y1 100.1 mm to (92.9, 89.7), turned to 45 degrees
- moved C15 94.9 mm to (94.5, 91.3), turned to -135 degrees
- moved C11 93.7 mm to (98.0, 74.8), turned to 135 degrees
- moved C3 92.3 mm to (102.2, 74.8), turned to 45 degrees
- moved C6 88.0 mm to (91.3, 91.3), turned to 135 degrees
- moved C9 86.7 mm to (95.4, 85.0), turned to -135 degrees
- moved C4 86.6 mm to (104.0, 76.7), turned to 45 degrees
- moved C12 80.8 mm to (106.2, 81.4), turned to 45 degrees
- moved C2 79.1 mm to (109.1, 77.1), turned to -90 degrees
- moved F1 75.4 mm to (125.8, 76.6)
- moved C10 74.6 mm to (95.2, 77.8), turned to 135 degrees
- moved C1 72.7 mm to (113.9, 77.1), turned to -90 degrees
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- renumbered C13 to C10, C14 to C12
Connections:
- J2 pad 1: unconnected-(J2-Pad1) -> GP23
- J2 pad 10: unconnected-(J2-Pad10) -> GP14
- J2 pad 11: unconnected-(J2-Pad11) -> GP13
- J2 pad 12: unconnected-(J2-Pad12) -> GP12
- J2 pad 13: unconnected-(J2-Pad13) -> GP11
- J2 pad 14: unconnected-(J2-Pad14) -> GP10
- J2 pad 2: unconnected-(J2-Pad2) -> GP22
- J2 pad 3: unconnected-(J2-Pad3) -> GP21
- J2 pad 4: unconnected-(J2-Pad4) -> GP20
- J2 pad 5: unconnected-(J2-Pad5) -> GP19
- J2 pad 6: unconnected-(J2-Pad6) -> GP18
- J2 pad 7: unconnected-(J2-Pad7) -> GP17
- J2 pad 8: unconnected-(J2-Pad8) -> GP16
- J2 pad 9: unconnected-(J2-Pad9) -> GP15
- J5 pad 1: unconnected-(J5-Pad1) -> GP29
- J5 pad 2: unconnected-(J5-Pad2) -> GP28
- J5 pad 3: unconnected-(J5-Pad3) -> GP27
- J5 pad 4: unconnected-(J5-Pad4) -> GP26
- J5 pad 5: unconnected-(J5-Pad5) -> GP25
- J5 pad 6: unconnected-(J5-Pad6) -> GP24
- R1 pad 1: Net-(J1-PadA5) -> GND
- R1 pad 2: GND -> Net-(J3-PadA5)
- R2 pad 1: Net-(J1-PadB5) -> GND
- R2 pad 2: GND -> Net-(J3-PadB5)
- SW7 pad 1: unconnected-(SW7-Pad1) -> GP23
- SW7 pad 2: unconnected-(SW7-Pad2) -> Net-(D1-Pad2)
- SW8 pad 1: unconnected-(SW8-Pad1) -> Net-(SW8-Pad1)
- SW8 pad 2: unconnected-(SW8-Pad2) -> GP0
- SW9 pad 1: unconnected-(SW9-Pad1) -> Net-(SW9-Pad1)
- SW9 pad 2: unconnected-(SW9-Pad2) -> GP1
- U1 pad 11: unconnected-(U1-Pad11) -> GP8
- U1 pad 12: unconnected-(U1-Pad12) -> GP9
- U1 pad 13: unconnected-(U1-Pad13) -> GP10
- U1 pad 14: unconnected-(U1-Pad14) -> GP11
- U1 pad 15: unconnected-(U1-Pad15) -> GP12
- U1 pad 16: unconnected-(U1-Pad16) -> GP13
- U1 pad 17: unconnected-(U1-Pad17) -> GP14
- U1 pad 18: unconnected-(U1-Pad18) -> GP15
- U1 pad 2: unconnected-(U1-Pad2) -> GP0
- U1 pad 27: unconnected-(U1-Pad27) -> GP16
- U1 pad 28: unconnected-(U1-Pad28) -> GP17
- U1 pad 29: unconnected-(U1-Pad29) -> GP18
- U1 pad 3: unconnected-(U1-Pad3) -> GP1
- U1 pad 30: unconnected-(U1-Pad30) -> GP19
- U1 pad 31: unconnected-(U1-Pad31) -> GP20
- U1 pad 32: unconnected-(U1-Pad32) -> GP21
- U1 pad 34: unconnected-(U1-Pad34) -> GP22
- U1 pad 35: unconnected-(U1-Pad35) -> GP23
- U1 pad 36: unconnected-(U1-Pad36) -> GP24
- U1 pad 37: unconnected-(U1-Pad37) -> GP25
- U1 pad 38: unconnected-(U1-Pad38) -> GP26
- U1 pad 39: unconnected-(U1-Pad39) -> GP27
- U1 pad 4: unconnected-(U1-Pad4) -> GP2
- U1 pad 40: unconnected-(U1-Pad40) -> GP28
- U1 pad 41: unconnected-(U1-Pad41) -> GP29
- U1 pad 5: unconnected-(U1-Pad5) -> GP3
- U1 pad 6: unconnected-(U1-Pad6) -> GP4
- U1 pad 7: unconnected-(U1-Pad7) -> GP5
- U1 pad 8: unconnected-(U1-Pad8) -> GP6
- U1 pad 9: unconnected-(U1-Pad9) -> GP7
- U3 pad 1: D- -> D+
- U3 pad 3: D+ -> unconnected-(U3-Pad3)
- U3 pad 5: VBUS -> +5V
- U3 pad 6: unconnected-(U3-Pad6) -> D-
Routing:
- net GND: track 0.00 -> 295.3 mm, vias 0 -> 26
- net +3V3: track 0.00 -> 86.4 mm, vias 0 -> 7
- net GP7: track 0.00 -> 57.3 mm, vias 0 -> 3
- net D-: track 0.00 -> 55.9 mm, vias 0 -> 2
- net D+: track 0.00 -> 54.8 mm, vias 0 -> 2
- net GP1: track 0.00 -> 51.8 mm, vias 0 -> 4
- net QSPI_SS: track 0.00 -> 48.4 mm, vias 0 -> 2
- net GP6: track 0.00 -> 39.6 mm, vias 0 -> 2
- net GP2: track 0.00 -> 39.3 mm
- net GP18: track 0.00 -> 38.9 mm, vias 0 -> 2
- net GP0: track 0.00 -> 38.8 mm, vias 0 -> 2
- net GP3: track 0.00 -> 37.5 mm, vias 0 -> 2
- net GP4: track 0.00 -> 36.7 mm, vias 0 -> 2
- net GP5: track 0.00 -> 34.6 mm, vias 0 -> 2
- net VBUS: track 0.00 -> 33.4 mm, vias 0 -> 1
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- added copper zone on B.Cu, net GND
- added copper zone on F.Cu, net GND
Other:
- board size 93.7 x 55.6 mm -> 55.6 x 31 mm
- board text added: "0"
- board text added: "1"
- board text added: "10"
- board text added: "11"
- board text added: "12"
- board text added: "13"
- board text added: "14"
- board text added: "15"
- board text added: "16"
- board text added: "17"
- board text added: "18"
- board text added: "19"
- board text added: "2"
- board text added: "20"
- board text added: "21"
- board text added: "22"
- board text added: "23"
- board text added: "23 0 1"
- board text added: "24"
- board text added: "25"
- board text added: "26"
- board text added: "27"
- board text added: "28"
- board text added: "29"
- board text added: "3"
- board text added: "4"
- board text added: "5"
- board text added: "5V"
- board text added: "6"
- board text added: "7"
- board text added: "8"
- board text added: "9"
- board text added: "D+"
- board text added: "D-"
- board text added: "GND"
- board text added: "Kiser Designs"
- board text added: "Piggyback"

Commit message: add gerbers
Routing:
- net GND: track 295.3 -> 306.9 mm
- net GP7: track 57.3 -> 59.3 mm
Changed lines of the file:
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@@
       (outputformat 1)
       (mirror false)
-      (drillshape 1)
+      (drillshape 0)
       (scaleselection 1)
-      (outputdirectory "")
+      (outputdirectory "Gerbers")
     )
   )
@@
     (pad "" thru_hole circle (at -3 -0.8) (size 0.6 0.6) (drill 0.4) (layers *.Cu))
     (pad "" smd roundrect (at 1.8 2) (size 0.75 1.2) (layers "B.Paste" "B.Mask") (roundrect_rratio 0.1666666667))
-    (pad "1" smd roundrect (at -1.8 2.2) (size 1 1.8) (layers "B.Cu") (roundrect_rratio 0.1666666667)
+    (pad "1" smd roundrect (at -1.8 2.2) (size 1 1.8) (layers "B.Cu") (roundrect_rratio 0.166667)
       (net 30 "+5V") (pinfunction "Pin_1") (pintype "passive"))
-    (pad "2" smd roundrect (at -0.6 2.2) (size 1 1.8) (layers "B.Cu") (roundrect_rratio 0.1666666667)
+    (pad "2" smd roundrect (at -0.6 2.2) (size 1 1.8) (layers "B.Cu") (roundrect_rratio 0.166667)
       (net 38 "D-") (pinfunction "Pin_2") (pintype "passive"))
-    (pad "3" smd roundrect (at 0.6 2.2) (size 1 1.8) (layers "B.Cu") (roundrect_rratio 0.1666666667)
+    (pad "3" smd roundrect (at 0.6 2.2) (size 1 1.8) (layers "B.Cu") (roundrect_rratio 0.166667)
       (net 37 "D+") (pinfunction "Pin_3") (pintype "passive"))
-    (pad "4" smd roundrect (at 1.8 2.2) (size 1 1.8) (layers "B.Cu") (roundrect_rratio 0.1666666667)
+    (pad "4" smd roundrect (at 1.8 2.2) (size 1 1.8) (layers "B.Cu") (roundrect_rratio 0.166667)
       (net 31 "GND") (pinfunction "Pin_4") (pintype "passive"))
     (pad "MP" smd roundrect (at 2.575 -1.5) (size 1.45 2) (layers "B.Cu") (roundrect_rratio 0.06896551724)
@@
   (segment (start 86.8 93.8) (end 90.2 90.4) (width 0.2) (layer "F.Cu") (net 31))
   (segment (start 130.2125 85.1625) (end 133.6125 85.1625) (width 0.2) (layer "F.Cu") (net 31))
+  (segment (start 130.96875 88.9) (end 134.525355 88.9) (width 0.2) (layer "F.Cu") (net 31))
   (segment (start 125.4125 75.40625) (end 126.20625 75.40625) (width 0.2) (layer "F.Cu") (net 31))
   (segment (start 124.4125 88.9625) (end 123.4125 89.9625) (width 0.2) (layer "F.Cu") (net 31))
@@
   (segment (start 93.33435 89.46565) (end 93.33435 87.428208) (width 0.2) (layer "F.Cu") (net 31))
   (segment (start 107.093934 79.293934) (end 107.093934 80.918198) (width 0.2) (layer "F.Cu") (net 31))
+  (segment (start 129.90625 89.9625) (end 130.96875 88.9) (width 0.2) (layer "F.Cu") (net 31))
+  (segment (start 134.525355 88.9) (end 134.556509 88.868846) (width 0.2) (layer "F.Cu") (net 31))
   (segment (start 134.842855 88.5825) (end 134.556509 88.868846) (width 0.2) (layer "F.Cu") (net 31))
   (segment (start 100.0125 80.9625) (end 97.0125 83.9625) (width 0.2) (layer "F.Cu") (net 31))
@@
   (segment (start 116.729346 77.879346) (end 119.730076 77.879346) (width 0.2) (layer "F.Cu") (net 31))
   (segment (start 100.09269 74.28231) (end 104.725654 74.28231) (width 0.2) (layer "F.Cu") (net 31))
+  (segment (start 123.4125 89.9625) (end 129.90625 89.9625) (width 0.2) (layer "F.Cu") (net 31))
   (via (at 94.385951 77.172827) (size 0.6) (drill 0.3) (layers "F.Cu" "B.Cu") (net 31))
   (via (at 106.290188 75.846844) (size 0.6) (drill 0.3) (layers "F.Cu" "B.Cu") (net 31))
@@
   (segment (start 102.4125 87.9625) (end 106.4125 91.9625) (width 0.2) (layer "B.Cu") (net 69))
   (segment (start 102.4125 85.342399) (end 102.4125 87.9625) (width 0.2) (layer "B.Cu") (net 69))
+  (segment (start 129.064054 92.1625) (end 130.396762 90.829792) (width 0.2) (layer "F.Cu") (net 70))
   (segment (start 126.4375 92.1625) (end 112.8125 92.1625) (width 0.2) (layer "F.Cu") (net 70))
   (segment (start 101.8125 91.1625) (end 111.0125 91.1625) (width 0.2) (layer "F.Cu") (net 70))
   (segment (start 112.8125 92.1625) (end 111.4125 90.7625) (width 0.2) (layer "F.Cu") (net 70))
+  (segment (start 126.4375 92.1625) (end 129.064054 92.1625) (width 0.2) (layer "F.Cu") (net 70))
   (segment (start 111.0125 91.1625) (end 111.4125 90.7625) (width 0.2) (layer "F.Cu") (net 70))
-  (segment (start 128 90.6) (end 126.4375 92.1625) (width 0.2) (layer "F.Cu") (net 70))
   (via (at 101.8125 91.1625) (size 0.6) (drill 0.3) (layers "F.Cu" "B.Cu") (net 70))
+  (via (at 130.396762 90.829792) (size 0.6) (drill 0.3) (layers "F.Cu" "B.Cu") (net 70))
   (via (at 111.4125 90.7625) (size 0.6) (drill 0.3) (layers "F.Cu" "B.Cu") (net 70))
-  (via (at 128 90.6) (size 0.6) (drill 0.3) (layers "F.Cu" "B.Cu") (net 70))
   (segment (start 107.874796 89.663287) (end 107.614297 89.402788) (width 0.2) (layer "B.Cu") (net 70))
   (segment (start 110.39375 90.4875) (end 109.569537 89.663287) (width 0.2) (layer "B.Cu") (net 70))
@@
   (segment (start 104.211139 86.064776) (end 103.706087 86.064776) (width 0.2) (layer "B.Cu") (net 70))
   (segment (start 111.4125 90.7625) (end 111.1375 90.4875) (width 0.2) (layer "B.Cu") (net 70))
+  (segment (start 130.396762 90.829792) (end 130.05447 90.4875) (width 0.2) (layer "B.Cu") (net 70))
   (segment (start 109.569537 89.663287) (end 107.874796 89.663287) (width 0.2) (layer "B.Cu") (net 70))
   (segment (start 121.0275 94.3625) (end 122.70875 96.04375) (width 0.2) (layer "B.Cu") (net 70))
   (segment (start 104.211139 86.064776) (end 104.975434 86.829071) (width 0.2) (layer "B.Cu") (net 70))
   (segment (start 110.39375 90.94375) (end 111.0125 91.5625) (width 0.2) (layer "B.Cu") (net 70))
-  (segment (start 129.44375 90.4875) (end 128.1125 90.4875) (width 0.2) (layer "B.Cu") (net 70))
-  (segment (start 128.1125 90.4875) (end 128 90.6) (width 0.2) (layer "B.Cu") (net 70))
+  (segment (start 130.05447 90.4875) (end 129.44375 90.4875) (width 0.2) (layer "B.Cu") (net 70))
   (segment (start 113.0125 86.29052) (end 111.4125 87.89052) (width 0.2) (layer "F.Cu") (net 71))
   (segment (start 101.4125 82.658044) (end 101.4125 81.9625) (width 0.2) (layer "F.Cu") (net 71))

Commit message: cost engineering
Parts:
- removed C15: 30p, Capacitor_SMD:C_0201_0603Metric
- removed SW1, SW10, SW11, SW12, SW13, SW14, SW15, SW2, SW3, SW5, SW6: MX_SW_solder, marbastlib-mx:SW_MX_1u
- removed Y1: Crystal_GND24_Small, Crystal:Crystal_SMD_2520-4Pin_2.5x2.0mm
- added Y2: Crystal_GND2_Small, Crystal:Resonator_SMD_Murata_CSTxExxV-3Pin_3.0x1.1mm, B.Cu at (93.7, 89.7)
- C1, C2: value 10u -> 1u; footprint Capacitor_SMD:C_0201_0603Metric -> Capacitor_SMD:C_0402_1005Metric
- C3, C5: footprint Capacitor_SMD:C_0201_0603Metric -> Capacitor_SMD:C_0402_1005Metric
- C6: value 30p -> 100n
- R1, R2, R3, R4, R5, R6, R8: footprint Resistor_SMD:R_0201_0603Metric -> Resistor_SMD:R_0402_1005Metric
- SWR1, SWR2: footprint Button_Switch_SMD:SW_SPST_B3U-1000P -> Button_Switch_SMD:SW_Push_SPST_NO_Alps_SKRK
- moved C6 12.7 mm to (102.6, 85.6), turned to -90 degrees
- moved R8 4.85 mm to (134.4, 78.5), turned to 0 degrees
- moved R4 1.61 mm to (106.4, 74.8), turned to 0 degrees
- moved C3 0.99 mm to (101.2, 74.8), turned to 0 degrees
- moved R5 0.89 mm to (106.4, 75.8), turned to 0 degrees
- moved C12 0.61 mm to (106.8, 81.6), turned to 0 degrees
- moved R6 0.57 mm to (93.0, 86.0)
- moved R3 0.47 mm to (87.7, 75.9)
- moved R1 0.19 mm to (126.0, 73.1)
- moved C5 0.19 mm to (102.6, 75.4)
- moved C1 0.14 mm to (114.0, 77.1)
- moved R7 0.11 mm to (129.7, 77.8)
- moved J3 0.11 mm to (127.8, 67.4)
- moved C2 0.10 mm to (109.0, 77.1)
Connections:
- C6 pad 1: GND -> +3V3
- C6 pad 2: Net-(C6-Pad2) -> GND
- R6 pad 1: Net-(C6-Pad2) -> Net-(R6-Pad1)
Routing:
- net Net-(C6-Pad2): track 4.97 -> 0.00 mm
- net Net-(R6-Pad1): track 0.00 -> 3.45 mm
- net Net-(SWR2-B): track 5.71 -> 2.59 mm
- net D-: track 55.9 -> 53.9 mm
- net XIN: track 9.01 -> 7.18 mm
- net GP18: track 38.9 -> 37.1 mm
- net d-: track 4.16 -> 5.60 mm
- net D+: track 54.8 -> 53.5 mm
- net +3V3: track 86.4 -> 87.6 mm
- net +5V: track 22.1 -> 21.1 mm
- net RUN: track 17.4 -> 18.4 mm
- net VBUS: track 33.4 -> 34.2 mm
- net d+: track 4.35 -> 5.19 mm
- net GND: track 306.9 -> 306.5 mm, vias 26 -> 27

Commit message: further cost reductions
Parts:
- removed C6: 100n, Capacitor_SMD:C_0201_0603Metric
- C10, C11, C12, C16, C7, C8, C9: footprint Capacitor_SMD:C_0201_0603Metric -> Capacitor_SMD:C_0402_1005Metric
- moved R5 0.82 mm to (107.2, 76.0)
- moved C10 0.80 mm to (94.4, 78.0), turned to 180 degrees
- moved C11 0.73 mm to (98.7, 74.8), turned to 180 degrees
- moved C7 0.61 mm to (106.0, 77.4)
- moved C8 0.30 mm to (94.6, 84.2)
Routing:
- net GND: track 306.5 -> 290.9 mm, vias 27 -> 26
- net +3V3: track 87.6 -> 85.5 mm
- net GP23: track 29.2 -> 30.1 mm
- net d+: track 5.19 -> 5.99 mm
- net RUN: track 18.4 -> 19.0 mm
