File: Piggyback_2_0/Piggyback_2_0.kicad_pcb (KiCad board)
At the start: 2 copper layers, 55.6 x 31 mm, 42 parts, among them J1 Conn_01x06_Female, J2 Conn_01x23_Female, J3 USB_C_Receptacle_USB2.0, J5 Conn_01x06_Female, SW7 MX_SW_solder, SW8 MX_SW_solder, SW9 MX_SW_solder, U1 RP2040TR7, U2 XC6206PxxxMR, U3 SRV05-4, U4 W25Q128JVS, Y2 Crystal_GND2_Small

Commit message: usb-spec crystal
Parts:
- moved C9 0.06 mm to (95.3, 84.9)
- moved C8 0.06 mm to (94.6, 84.1)
- turned Y2 to 180 degrees
Connections:
- Y2 pad 1: Net-(R6-Pad1) -> XIN
- Y2 pad 3: XIN -> Net-(R6-Pad1)
Changed lines of the file:
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@@
   )
   (footprint "Capacitor_SMD:C_0402_1005Metric" (layer "B.Cu")
-    (at 94.6125 84.1625 -135)
+    (at 94.558586 84.133235 -135)
     (descr "Capacitor SMD 0402 (1005 Metric), square (rectangular) end terminal, IPC_7351 nominal, (Body size source: IPC-SM-782 page 76, https://www.pcb-3d.com/wordpress/wp-content/uploads/ipc-sm-782a_amendment_1_and_2.pdf), generated with kicad-footprint-generator")
     (tags "capacitor")
@@
   )
   (footprint "Capacitor_SMD:C_0402_1005Metric" (layer "B.Cu")
-    (at 95.4 84.9625 -135)
+    (at 95.346086 84.933235 -135)
     (descr "Capacitor SMD 0402 (1005 Metric), square (rectangular) end terminal, IPC_7351 nominal, (Body size source: IPC-SM-782 page 76, https://www.pcb-3d.com/wordpress/wp-content/uploads/ipc-sm-782a_amendment_1_and_2.pdf), generated with kicad-footprint-generator")
     (tags "capacitor")
@@
   )
   (footprint "Crystal:Resonator_SMD_Murata_CSTxExxV-3Pin_3.0x1.1mm" (layer "B.Cu")
-    (at 93.6625 89.69375)
+    (at 93.6625 89.69375 180)
     (descr "SMD Resomator/Filter Murata CSTCE, https://www.murata.com/en-eu/products/productdata/8801162264606/SPEC-CSTNE16M0VH3C000R0.pdf")
     (tags "SMD SMT ceramic resonator filter")
@@
     (property "ki_keywords" "quartz ceramic resonator oscillator")
     (attr smd)
-    (fp_text reference "Y2" (at 0 2) (layer "B.SilkS")
+    (fp_text reference "Y2" (at 0 -2.38125) (layer "B.SilkS")
         (effects (font (size 1 1) (thickness 0.15)) (justify mirror))
     )
@@
     (fp_line (start 1.5 0.8) (end -1.5 0.8)
       (stroke (width 0.1) (type solid)) (layer "B.Fab"))
-    (pad "1" smd rect (at -1.2 0) (size 0.4 1.9) (layers "B.Cu" "B.Paste" "B.Mask")
-      (net 61 "Net-(R6-Pad1)") (pinfunction "1") (pintype "passive"))
-    (pad "2" smd rect (at 0 0) (size 0.4 1.9) (layers "B.Cu" "B.Paste" "B.Mask")
+    (pad "1" smd rect (at -1.2 0 180) (size 0.4 1.9) (layers "B.Cu" "B.Paste" "B.Mask")
+      (net 12 "XIN") (pinfunction "1") (pintype "passive"))
+    (pad "2" smd rect (at 0 0 180) (size 0.4 1.9) (layers "B.Cu" "B.Paste" "B.Mask")
       (net 9 "GND") (pinfunction "2") (pintype "passive"))
-    (pad "3" smd rect (at 1.2 0) (size 0.4 1.9) (layers "B.Cu" "B.Paste" "B.Mask")
-      (net 12 "XIN") (pinfunction "3") (pintype "passive"))
+    (pad "3" smd rect (at 1.2 0 180) (size 0.4 1.9) (layers "B.Cu" "B.Paste" "B.Mask")
+      (net 61 "Net-(R6-Pad1)") (pinfunction "3") (pintype "passive"))
     (model "${KICAD6_3DMODEL_DIR}/Crystal.3dshapes/Resonator_SMD_Murata_CSTxExxV-3Pin_3.0x1.1mm.wrl"
       (offset (xyz 0 0 0))
@@
   (via (at 90.2 90.2) (size 0.6) (drill 0.3) (layers "F.Cu" "B.Cu") (net 9))
   (via (at 117.4125 87.3625) (size 0.6) (drill 0.3) (layers "F.Cu" "B.Cu") (net 9))
+  (via (at 94.30569 85.187532) (size 0.6) (drill 0.3) (layers "F.Cu" "B.Cu") (net 9))
   (via (at 105.4125 76.1625) (size 0.6) (drill 0.3) (layers "F.Cu" "B.Cu") (net 9))
   (via (at 114.775 74.6) (size 0.6) (drill 0.3) (layers "F.Cu" "B.Cu") (net 9))
   (via (at 101.6 80.9625) (size 0.6) (drill 0.3) (layers "F.Cu" "B.Cu") (net 9))
   (via (at 121.2125 79.5625) (size 0.6) (drill 0.3) (layers "F.Cu" "B.Cu") (net 9))
-  (via (at 94.363957 85.32128) (size 0.6) (drill 0.3) (layers "F.Cu" "B.Cu") (net 9))
   (via (at 134.556509 88.868846) (size 0.6) (drill 0.3) (layers "F.Cu" "B.Cu") (net 9))
   (via (at 98.425 80.9625) (size 0.6) (drill 0.3) (layers "F.Cu" "B.Cu") (net 9))
@@
   (segment (start 93.521171 77.9625) (end 93.516974 77.966697) (width 0.2) (layer "B.Cu") (net 9))
   (segment (start 123.34525 74.22975) (end 124.402412 74.22975) (width 0.2) (layer "B.Cu") (net 9))
+  (segment (start 94.921561 85.187532) (end 94.30569 85.187532) (width 0.2) (layer "B.Cu") (net 9))
   (segment (start 121.6875 74.5625) (end 121.5925 74.6575) (width 0.2) (layer "B.Cu") (net 9))
   (segment (start 93.6625 88.114039) (end 93.436634 87.888173) (width 0.2) (layer "B.Cu") (net 9))
@@
   (segment (start 114.775 74.6) (end 115.975 74.6) (width 0.2) (layer "B.Cu") (net 9))
   (segment (start 130.96875 73.81875) (end 130.902639 73.81875) (width 0.2) (layer "B.Cu") (net 9))
-  (segment (start 95.07872 85.32128) (end 94.363957 85.32128) (width 0.2) (layer "B.Cu") (net 9))
   (segment (start 122.798593 81.173692) (end 122.233397 81.173692) (width 0.2) (layer "B.Cu") (net 9))
   (segment (start 106.557073 77.464573) (end 106.4925 77.4) (width 0.2) (layer "B.Cu") (net 9))
@@
   (segment (start 91.507524 91.692476) (end 91.507524 91.507524) (width 0.2) (layer "B.Cu") (net 9))
   (segment (start 107.097865 80.931965) (end 106.966432 80.800532) (width 0.2) (layer "B.Cu") (net 9))
-  (segment (start 94.573726 84.626274) (end 94.363957 84.836043) (width 0.2) (layer "B.Cu") (net 9))
   (segment (start 93.33435 87.855815) (end 93.33435 88.103592) (width 0.2) (layer "B.Cu") (net 9))
   (segment (start 93.6625 91.507524) (end 94.229976 91.507524) (width 0.2) (layer "B.Cu") (net 9))
@@
   (segment (start 116.969126 87.805874) (end 117.4125 87.3625) (width 0.2) (layer "B.Cu") (net 9))
   (segment (start 96.919607 85.469607) (end 97.0125 85.5625) (width 0.2) (layer "B.Cu") (net 9))
-  (segment (start 94.363957 84.836043) (end 94.363957 85.32128) (width 0.2) (layer "B.Cu") (net 9))
+  (segment (start 94.219175 84.472646) (end 94.363957 84.617428) (width 0.2) (layer "B.Cu") (net 9))
   (segment (start 129.70125 73.125) (end 130.208889 73.125) (width 0.2) (layer "B.Cu") (net 9))
+  (segment (start 94.219175 84.472646) (end 94.219175 85.101017) (width 0.2) (layer "B.Cu") (net 9))
   (segment (start 120.6125 78.5625) (end 120.6125 77.582224) (width 0.4) (layer "B.Cu") (net 9))
   (segment (start 101.6925 74.7625) (end 102.647572 74.7625) (width 0.2) (layer "B.Cu") (net 9))
@@
   (segment (start 120.319849 77.289573) (end 120.4125 77.382225) (width 0.2) (layer "B.Cu") (net 9))
   (segment (start 96.8125 86.3625) (end 97.0125 86.1625) (width 0.2) (layer "B.Cu") (net 9))
+  (segment (start 95.006675 85.272646) (end 94.921561 85.187532) (width 0.2) (layer "B.Cu") (net 9))
   (segment (start 102.647572 74.7625) (end 102.615048 74.7625) (width 0.2) (layer "B.Cu") (net 9))
   (segment (start 93.6625 89.69375) (end 93.6625 91.507524) (width 0.2) (layer "B.Cu") (net 9))
   (segment (start 98.290695 84.098519) (end 96.919607 85.469607) (width 0.2) (layer "B.Cu") (net 9))
   (segment (start 124.38875 71.51375) (end 123.47375 70.59875) (width 0.2) (layer "B.Cu") (net 9))
+  (segment (start 94.219175 85.101017) (end 94.30569 85.187532) (width 0.2) (layer "B.Cu") (net 9))
   (segment (start 114.6125 77.7625) (end 119.8125 82.9625) (width 0.2) (layer "F.Cu") (net 10))
   (segment (start 126.8125 80.5625) (end 125.2125 82.1625) (width 0.2) (layer "F.Cu") (net 10))
@@
   (segment (start 96.876481 79.240695) (end 95.66206 78.026274) (width 0.2) (layer "B.Cu") (net 10))
   (segment (start 103.660589 77.139411) (end 102.987061 77.139411) (width 0.2) (layer "B.Cu") (net 10))
-  (segment (start 95.918431 84.773726) (end 95.626274 84.773726) (width 0.2) (layer "B.Cu") (net 10))
+  (segment (start 96.098332 84.593824) (end 96.696078 83.996078) (width 0.2) (layer "B.Cu") (net 10))
   (segment (start 100.070847 76.695111) (end 100.602934 76.695111) (width 0.2) (layer "B.Cu") (net 10))
   (segment (start 97.293934 79.658148) (end 96.876481 79.240695) (width 0.2) (layer "B.Cu") (net 10))
   (segment (start 94.956274 78.026274) (end 94.8925 77.9625) (width 0.2) (layer "B.Cu") (net 10))
-  (segment (start 97.442167 83.24999) (end 95.918431 84.773726) (width 0.2) (layer "B.Cu") (net 10))
   (segment (start 99.422066 76.695111) (end 100.070847 76.695111) (width 0.2) (layer "B.Cu") (net 10))
   (segment (start 102.987061 77.139411) (end 102.987061 77.425071) (width 0.2) (layer "B.Cu") (net 10))
@@
   (segment (start 108.888198 76.7625) (end 109.0125 76.638198) (width 0.2) (layer "B.Cu") (net 10))
   (segment (start 100.070847 77.341285) (end 100.070847 76.695111) (width 0.2) (layer "B.Cu") (net 10))
+  (segment (start 95.685497 84.593824) (end 96.098332 84.593824) (width 0.2) (layer "B.Cu") (net 10))
   (segment (start 121.064266 81.813692) (end 120.779126 81.528552) (width 0.2) (layer "B.Cu") (net 10))
   (segment (start 97.973959 82.718198) (end 97.442167 83.24999) (width 0.2) (layer "B.Cu") (net 10))
@@
   (segment (start 97.293934 80.118198) (end 97.293934 79.718198) (width 0.2) (layer "B.Cu") (net 10))
   (segment (start 104.813262 76.7625) (end 108.888198 76.7625) (width 0.2) (layer "B.Cu") (net 10))
+  (segment (start 97.442167 83.24999) (end 96.696078 83.996078) (width 0.2) (layer "B.Cu") (net 10))
   (segment (start 102.987061 77.425071) (end 102.893934 77.518198) (width 0.2) (layer "B.Cu") (net 10))
   (segment (start 97.973959 82.718198) (end 97.973959 82.398223) (width 0.2) (layer "B.Cu") (net 10))
