File: Piggyback_2_0/Piggyback_2_0.kicad_sch (KiCad schematic)
At the start: 53 parts, among them J1 Conn_01x06_Female, J2 Conn_01x23_Female, J5 Conn_01x06_Female, SW1 MX_SW_solder, SW10 MX_SW_solder, SW11 MX_SW_solder, SW12 MX_SW_solder, SW13 MX_SW_solder, SW14 MX_SW_solder, SW15 MX_SW_solder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

Commit message: cost engineering
Parts:
- removed C15: 30p, Capacitor_SMD:C_0201_0603Metric, symbol Device:C_Small
- removed Y1: Crystal_GND24_Small, Crystal:Crystal_SMD_2520-4Pin_2.5x2.0mm, symbol Device:Crystal_GND24_Small
- added Y2: Crystal_GND2_Small, Crystal:Resonator_SMD_Murata_CSTxExxV-3Pin_3.0x1.1mm, symbol Device:Crystal_GND2_Small
- C1, C2: value 10u -> 1u; footprint Capacitor_SMD:C_0201_0603Metric -> Capacitor_SMD:C_0402_1005Metric
- C3, C5: footprint Capacitor_SMD:C_0201_0603Metric -> Capacitor_SMD:C_0402_1005Metric
- C6: value 30p -> 100n
- J3: renamed from J?; footprint (none) -> Connector_USB:USB_C_Receptacle_HRO_TYPE-C-31-M-12
- R1, R2: renamed from R?; footprint Resistor_SMD:R_0201_0603Metric -> Resistor_SMD:R_0402_1005Metric
- R3, R4, R5, R6, R8: footprint Resistor_SMD:R_0201_0603Metric -> Resistor_SMD:R_0402_1005Metric
- SWR1, SWR2: footprint Button_Switch_SMD:SW_SPST_B3U-1000P -> Button_Switch_SMD:SW_Push_SPST_NO_Alps_SKRK
Connections:
- net +3V3: now also C6.1
- net GND: now also C6.2, Y2.2; no longer C6.1
- net XIN: now also Y2.3
- net at R6.1: now also Y2.1; no longer C6.2

Commit message: further cost reductions
Parts:
- removed C6: 100n, Capacitor_SMD:C_0201_0603Metric, symbol Device:C_Small
- C10, C11, C12, C16, C7, C8, C9: footprint Capacitor_SMD:C_0201_0603Metric -> Capacitor_SMD:C_0402_1005Metric
Changed lines of the file:
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@@
   (junction (at 200.025 153.035) (diameter 0) (color 0 0 0 0)
   )
-  (junction (at 216.535 147.955) (diameter 0) (color 0 0 0 0)
-  )
   (junction (at 19.05 109.22) (diameter 0) (color 0 0 0 0)
   )
@@
     (stroke (width 0) (type default))
   )
-  (wire (pts (xy 216.535 147.955) (xy 224.79 147.955))
-    (stroke (width 0) (type default))
-  )
   (wire (pts (xy 40.005 25.4) (xy 43.815 25.4))
     (stroke (width 0) (type default))
@@
   )
   (wire (pts (xy 24.765 104.14) (xy 26.035 104.14))
-    (stroke (width 0) (type default))
-  )
-  (wire (pts (xy 216.535 153.035) (xy 224.79 153.035))
     (stroke (width 0) (type default))
   )
@@
       (effects (font (size 1.27 1.27)) (justify left))
     )
-    (property "Footprint" "Capacitor_SMD:C_0201_0603Metric" (at 173.355 150.495 0)
+    (property "Footprint" "Capacitor_SMD:C_0402_1005Metric" (at 173.355 150.495 0)
       (effects (font (size 1.27 1.27)) hide)
     )
@@
       (effects (font (size 1.27 1.27)) (justify left))
     )
-    (property "Footprint" "Capacitor_SMD:C_0201_0603Metric" (at 181.61 150.495 0)
+    (property "Footprint" "Capacitor_SMD:C_0402_1005Metric" (at 181.61 150.495 0)
       (effects (font (size 1.27 1.27)) hide)
     )
@@
       (effects (font (size 1.27 1.27)) (justify left))
     )
-    (property "Footprint" "Capacitor_SMD:C_0201_0603Metric" (at 191.77 150.495 0)
+    (property "Footprint" "Capacitor_SMD:C_0402_1005Metric" (at 191.77 150.495 0)
       (effects (font (size 1.27 1.27)) hide)
     )
@@
       (effects (font (size 1.27 1.27)) (justify left))
     )
-    (property "Footprint" "Capacitor_SMD:C_0201_0603Metric" (at 200.025 150.495 0)
+    (property "Footprint" "Capacitor_SMD:C_0402_1005Metric" (at 200.025 150.495 0)
       (effects (font (size 1.27 1.27)) hide)
     )
@@
         (path "/b12e0c4a-97f3-4d57-8489-3c2627093953"
           (reference "C10") (unit 1)
-        )
-      )
-    )
-  )
-  (symbol (lib_id "Device:C_Small") (at 224.79 150.495 0) (unit 1)
-    (in_bom yes) (on_board yes) (dnp no) (fields_autoplaced)
-    (property "Reference" "C6" (at 227.1141 149.5928 0)
-      (effects (font (size 1.27 1.27)) (justify left))
-    )
-    (property "Value" "100n" (at 227.1141 152.3679 0)
-      (effects (font (size 1.27 1.27)) (justify left))
-    )
-    (property "Footprint" "Capacitor_SMD:C_0201_0603Metric" (at 224.79 150.495 0)
-      (effects (font (size 1.27 1.27)) hide)
-    )
-    (property "Datasheet" "~" (at 224.79 150.495 0)
-      (effects (font (size 1.27 1.27)) hide)
-    )
-    (pin "1")
-    (pin "2")
-    (instances
-      (project "Piggyback_2_0"
-        (path "/b12e0c4a-97f3-4d57-8489-3c2627093953"
-          (reference "C6") (unit 1)
         )
       )
@@
       (effects (font (size 1.27 1.27)) (justify left))
     )
-    (property "Footprint" "Capacitor_SMD:C_0201_0603Metric" (at 155.575 158.75 0)
+    (property "Footprint" "Capacitor_SMD:C_0402_1005Metric" (at 155.575 158.75 0)
       (effects (font (size 1.27 1.27)) hide)
     )
@@
       (effects (font (size 1.27 1.27)) (justify left))
     )
-    (property "Footprint" "Capacitor_SMD:C_0201_0603Metric" (at 216.535 150.495 0)
+    (property "Footprint" "Capacitor_SMD:C_0402_1005Metric" (at 216.535 150.495 0)
       (effects (font (size 1.27 1.27)) hide)
     )
@@
       (effects (font (size 1.27 1.27)) (justify left))
     )
-    (property "Footprint" "Capacitor_SMD:C_0201_0603Metric" (at 208.28 150.495 0)
-      (effects (font (size 1.27 1.27)) hide)
-    )
+    (property "Footprint" "Capacitor_SMD:C_0402_1005Metric" (at 208.28 150.495 0)
+      (effects (font (size 1.27 1.27)) hide)
+    )

Commit message: usb-spec crystal
Connections:
- net XIN: now also Y2.1; no longer Y2.3
- net at R6.1: now also Y2.3; no longer Y2.1
Changed lines of the file:
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@@
     )
   )
-  (symbol (lib_id "Device:Crystal_GND2_Small") (at 128.905 149.225 270) (unit 1)
-    (in_bom yes) (on_board yes) (dnp no) (fields_autoplaced)
+  (symbol (lib_id "Device:Crystal_GND2_Small") (at 128.905 149.225 270) (mirror x) (unit 1)
+    (in_bom yes) (on_board yes) (dnp no)
     (property "Reference" "Y2" (at 132.08 148.59 90)
       (effects (font (size 1.27 1.27)) (justify left))
     )
-    (property "Value" "Crystal_GND2_Small" (at 132.08 151.13 90)
+    (property "Value" "Crystal_GND2_Small" (at 132.08 150.495 90)
       (effects (font (size 1.27 1.27)) (justify left))
     )

Commit message: add piggyback 3
Parts:
- removed SW4: MX_SW_solder, marbastlib-mx:SW_MX_1u, symbol marbastlib-mx:MX_SW_solder
- removed Y2: Crystal_GND2_Small, Crystal:Resonator_SMD_Murata_CSTxExxV-3Pin_3.0x1.1mm, symbol Device:Crystal_GND2_Small
- added C15, C6: 30p, Capacitor_SMD:C_0201_0603Metric, symbol Device:C_Small
- added Y1: Crystal_GND24_Small, Crystal:Crystal_SMD_2520-4Pin_2.5x2.0mm, symbol Device:Crystal_GND24_Small
- C1, C2: value 1u -> 10u; footprint Capacitor_SMD:C_0402_1005Metric -> Capacitor_SMD:C_0201_0603Metric
- C10, C11, C12, C16, C3, C5, C7, C8, C9: footprint Capacitor_SMD:C_0402_1005Metric -> Capacitor_SMD:C_0201_0603Metric
- R1, R2, R3, R4, R5, R6, R8: footprint Resistor_SMD:R_0402_1005Metric -> Resistor_SMD:R_0201_0603Metric
- SWR1, SWR2: footprint Button_Switch_SMD:SW_Push_SPST_NO_Alps_SKRK -> Button_Switch_SMD:SW_SPST_B3U-1000P
Connections:
- net GND: now also C15.2, C6.1, Y1.2, Y1.4
- net XIN: now also C15.1, Y1.3
- net at R6.1: now also C6.2, Y1.1
